Commit message: Add support for KUKA LBR IIWA 14 R820 robot with kinematics, joint limits, physical and visual parameters

File: urdf/inc/kuka_joint_control.xacro (robot description, xacro)
@@ -4,5 +4,5 @@
     params="
     tf_prefix
-    initial_positions:=${dict(joint_1=0.0,joint_2=-1.57,joint_3=0.0,joint_4=-1.57,joint_5=0.0,joint_6=0.0)}
+    initial_positions:=${dict(joint_1=0.0,joint_2=-1.57,joint_3=0.0,joint_4=-1.57,joint_5=0.0,joint_6=0.0,joint_7=0.0)}
     dof:=6
     ">
@@ -47,5 +47,5 @@
         <command_interface name="position" />
         <state_interface name="position">
-          <param name="initial_value">0.0</param>
+          <param name="initial_value">${initial_positions['joint_7']}</param>
         </state_interface>
       </joint>

File: urdf/kuka.urdf.xacro (robot description, xacro)
@@ -3,6 +3,4 @@
   <!-- robot name parameter -->
   <xacro:arg name="name" default="kuka" />
-  <!-- robot degree of freedom -->
-  <xacro:property name="dof" default="6" />
   <!-- import main macro -->
   <xacro:include filename="$(find kuka_robot_descriptions)/urdf/kuka_macro.xacro" />
@@ -21,4 +19,6 @@
   -->
   <xacro:arg name="kuka_type" default="kr6x" />
+  <!-- robot degree of freedom -->
+  <xacro:arg name="dof" default="6" />
   <!-- parameters for the robot -->
   <xacro:arg name="tf_prefix" default="" />
@@ -42,4 +42,5 @@
     name="$(arg name)"
     tf_prefix="$(arg tf_prefix)"
+    dof="$(arg dof)"
     parent="world"
     use_fake_hardware="$(arg use_fake_hardware)"
@@ -51,5 +52,4 @@
     client_port="$(arg client_port)"
     force_abs_paths="$(arg force_abs_paths)"
-    degrees_of_freedom="$(arg dof)"
   >
     <origin xyz="0 0 0" rpy="0 0 0" />          <!-- position robot in the world -->

File: urdf/kuka_macro.xacro (robot description, xacro)
@@ -25,4 +25,5 @@
     name
     tf_prefix
+    dof
     parent
     *origin
@@ -35,5 +36,4 @@
     visual_parameters_file
     force_abs_paths:=false
-    degrees_of_freedom
     ">
     <xacro:kuka_ros2_control
@@ -43,7 +43,7 @@
       client_port="${client_port}"
       use_fake_hardware="${use_fake_hardware}"
-      dof="${degrees_of_freedom}"
+      dof="${dof}"
     />
-    <xacro:kuka_arm_transmission tf_prefix="${tf_prefix}" dof="${degrees_of_freedom}" />
+    <xacro:kuka_arm_transmission tf_prefix="${tf_prefix}" dof="${dof}" />
     <!-- Load configuration data from the provided .yaml files -->
     <xacro:read_model_data
@@ -53,5 +53,5 @@
       visual_parameters_file="${visual_parameters_file}"
       force_abs_paths="${force_abs_paths}"
-      dof="${degrees_of_freedom}"
+      dof="${dof}"
     />
     <!-- Links -main serial chain -->
@@ -190,5 +190,5 @@
     </link>
     <!-- Link-7 -->
-    <xacro:if value="${degrees_of_freedom == 7}">
+    <xacro:if value="${dof == 7}">
       <link name="${tf_prefix}link_7">
         <visual>
@@ -278,5 +278,5 @@
     </joint>
     <!-- Joint-7 -->
-    <xacro:if value="${degrees_of_freedom == 7}">
+    <xacro:if value="${dof == 7}">
       <joint name="${tf_prefix}joint_7" type="revolute">
         <parent link="${tf_prefix}link_6" />
@@ -292,5 +292,5 @@
     <!-- ROS base_link to KUKA $ROBROOT coordinate system transform -->
     <link name="${tf_prefix}base" />
-    <joint name="${tf_prefix}base_link-base" type="fixed">
+    <joint name="${tf_prefix}base_link-base_joint" type="fixed">
       <origin xyz="0 0 0" rpy="0 0 0" />
       <parent link="${tf_prefix}base_link" />
@@ -298,5 +298,5 @@
     </joint>
     <!-- ROS-Industrial 'flange' frame - attachment point for EEF models -->
-    <xacro:if value="${degrees_of_freedom == 7}">
+    <xacro:if value="${dof == 7}">
       <link name="${tf_prefix}flange" />
       <joint name="${tf_prefix}joint_7-flange" type="fixed">
@@ -306,5 +306,5 @@
       </joint>
     </xacro:if>
-    <xacro:if value="${degrees_of_freedom == 6}">
+    <xacro:if value="${dof == 6}">
       <link name="${tf_prefix}flange" />
       <joint name="${tf_prefix}joint_6-flange" type="fixed">

File: urdf/ros2_control.xacro (robot description, xacro)
@@ -6,9 +6,9 @@
     name
     tf_prefix
-    initial_positions:=${dict(joint_1=0.0,joint_2=-1.57,joint_3=0.0,joint_4=-1.57,joint_5=0.0,joint_6=0.0)}
+    initial_positions:=${dict(joint_1=0.0,joint_2=-1.57,joint_3=0.0,joint_4=-1.57,joint_5=0.0,joint_6=0.0,joint_7=0.0)}
     client_ip
     client_port
     use_fake_hardware
-    dof:=6
+    dof
     ">
     <ros2_control name="${name}" type="system">
